File: hardware/kicad/monitors.kicad_sch (KiCad schematic)
At the start: 27 parts, among them U1301 MCP3208-BI/SL, U1302 MCP9700AT-E/TT

Commit message: feat(hardware)!: draw draft A1 of the schematic around a Pico 2
A Raspberry Pi Pico 2 on two 1x20 sockets replaces the ESP32-S3
development board, the programmable logic device and the buffer
between the two boards (D-39 to D-43 of the specification). The former
interface and range logic sheets become two new ones:

- Controller: the Pico 2, the diodes that join its USB supply and the
  5 V rail of the carrier, resistor arrays in the SPI and acquisition
  lines, a reset button and a console header.
- Side Data: two shift registers that take the range, the status
  signals and the eight logic inputs with every sample.

The DUT connects through a 1x4 pin header and a lever terminal block
in parallel, both GND, VIN, VOUT, GND, and the logic port is a 1x10
header with VCC, GND, D7 to D0: the pin order of the PPK2 (D-44). A
solder jumper selects the supply of the DUT side of the level
translator. A transistor at the driver of the ampere switch holds it
open while VIN is above 5.5 V.

Reference designators are numbered as the annotation tool of KiCad
does by default (D-45). The numbering touches every sheet, so these
changes come in one commit. The symbol and the socket footprint of
the ESP32-S3 board leave the project library; the Pico 2 uses the
symbol and the footprint of the KiCad library.

The electrical rules check reports no errors and no warnings. The
parts stay candidates, and no program for the PIO blocks exists yet.

BREAKING CHANGE: the pins of the controller follow the new pin map of
section 5 of the specification.
Parts:
- renumbered C1301 to C84, C1302 to C85, C1303 to C86, C1304 to C87, C1305 to C88, C1306 to C89, C1307 to C90, C1308 to C91, C1309 to C92, C1310 to C93, C1311 to C94, C1312 to C95, R1301 to R67, R1303 to R68, R1305 to R69, R1307 to R70, R1308 to R71, R1309 to R72, R1310 to R73, R1312 to R74, R1302 to R75, R1304 to R76, R1306 to R77, R1311 to R78, R1313 to R79, U1302 to U30, U1301 to U31
Connections:
- net SPI_MISO renamed C_MISO
Other:
- note added: "CH0 VOUT_BUF x 0.4545 CH1 VIN x 0.0833 CH2 +5V x 0.4545 CH3 CC1 CH4 CC2 CH5 0.5 V + 10 mV/K CH6 +12V_A x 0.1754 CH7 (-4V_A + 2 x VREF) / 3 U30 sits next to the linear regulator."
- note removed: "CH0 VOUT_BUF x 0.4545 CH1 VIN x 0.0833 CH2 +5V x 0.4545 CH3 CC1 CH4 CC2 CH5 0.5 V + 10 mV/K CH6 +12V_A x 0.1754 CH7 (-4V_A + 2 x VREF) / 3 U1302 sits next to the linear regulator."
