File: hardware/kicad/power-profiler-carrier.kicad_pcb (KiCad board)
At the start: 4 copper layers, 150 x 100 mm, 425 parts, among them J1 Debug UART, J2 USB-C power, J3 DUT, J4 DUT wires, J5 Logic port, Q1 BSS138, Q10 IRLML0030, Q11 IRLML0030, Q12 IRLML0030, Q13 IRLML0030, Q14 CSD17577Q3A, Q15 CSD17577Q3A, Q16 CSD17577Q3A, Q2 BSS138, Q3 BSS138, Q4 CSD17577Q3A, Q5 CSD17577Q3A, Q6 BC847B, Q7 BC847B, Q8 CSD17577Q3A, Q9 CSD17577Q3A, SW1 RESET, U1 Raspberry Pi Pico 2, U10 LMR62014XMF, U11 LM27761DSG, U12 REF5025AID, U13 LT3042EMSE, U14 MCP6569-E/SL, U15 MCP4921-E/SN, U16 TPS63020DSJ, U17 OPA197IDBV, U18 LT3080EDD, U19 OPA365AIDBV, U2 TPD4E1U06DBVR, U20 TC4427EOA, U21 MCP6561T-E/OT, U22 TC4427EOA, U23 TC4427EOA, U24 MUX509IPWR, U25 OPA197IDBV, U26 OPA197IDBV, U27 AD8421ARZ, U28 OPA365AIDBV, U29 OPA365AIDBV, U3 TPS259621DDAR, U30 ADS8860IDGS, U31 MCP6562-E/SN, U32 MCP6561T-E/OT, U33 SN74LV165ADR, U34 SN74LV165ADR, U35 TPD4E1U06DBVR, U36 TPD4E1U06DBVR, U37 TPD4E1U06DBVR, U38 SN74LVC8T245PW, U39 MCP9700AT-E/TT, U4 TPS259621DDAR, U40 MCP3208-BI/SL, U5 TPS2116DRLR, U6 TPS3808G01DBVR, U7 LP5907MFX-3.3, U8 LP5907MFX-3.3, U9 803 type, 3.08 V

Commit message: feat(hardware): review the layout of the carrier board
The autorouted board of draft A2 had 28 of its 984 connections open
and none of the copper that an autorouter does not draw. The layout is
now reviewed against section 10 of the specification:

- every connection is routed;
- the 1 A path is pours, with the supply band doubled on the bottom
  layer: 19.5 squares in source mode and 23.3 squares in ampere mode
  against the limit of 30;
- the measured node has its guard and the Kelvin lines of the four
  shunts, and no track on the bottom layer under the shield can; the
  surface leakage into it is 5.1 nA against a budget of 10 nA;
- the switch nodes and the output copper of the converters are pours,
  the 5 V rail is a pour on the second inner layer, and the reference
  leaves its pin as a star;
- ground fills on the second inner layer and on the bottom layer, with
  thermal reliefs on the through-hole ground pads.

The rule file now states every spacing that the layout needs (D-87):
the exemption near pins applies on the top layer only, and the
spacings against leakage along a surface apply on both outer layers.
The design rules check reports no violation, no unconnected pad, no
footprint error and no difference from the schematic.

Every figure is calculated from the drawn copper. Nothing is built or
measured, and no person has reviewed the board in the KiCad editor
yet.

The board file also carries the name of the project in the text on its
silkscreen and in its title block: "Open Power Profiler - Carrier
Board".
Parts:
- moved TP38 11.2 mm to (182.2, 106.8)
- moved D21 8.56 mm to (182.2, 100.5)
- moved R90 2.75 mm to (168.0, 131.6)
- moved R120 2.64 mm to (177.3, 96.9)
- moved TP7 2.55 mm to (80.8, 102.5)
- moved C74 2.50 mm to (182.1, 97.4)
- moved D20 2.50 mm to (178.2, 94.3)
- moved R115 2.50 mm to (173.5, 93.8), turned to 90 degrees
- moved R116 2.50 mm to (175.2, 93.8)
- moved R117 2.50 mm to (181.3, 94.9)
- moved TP37 2.50 mm to (183.8, 95.0)
- moved TP5 2.20 mm to (80.8, 105.2)
- moved TP36 1.97 mm to (171.3, 117.7)
- moved C76 1.62 mm to (142.6, 97.2), turned to 0 degrees
- moved R107 1.50 mm to (157.1, 113.2)
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Routing:
- net VREF: track 256.2 -> 538.3 mm, vias 7 -> 21
- net /Monitors/VOUT_BUF: track 63.3 -> 267.2 mm, vias 2 -> 11
- net /Path Switching/SUPPLY: track 123.5 -> 64.4 mm, vias 4 -> 34
- net Net-(U24-S4A): track 0.00 -> 46.3 mm, vias 0 -> 2
- net Net-(C42-Pad1): track 55.2 -> 12.0 mm, vias 2 -> 8
- net +13V5: track 77.2 -> 114.3 mm
- net Net-(D21-K): track 48.8 -> 18.7 mm, vias 2 -> 0
- net Net-(D13-K): track 6.76 -> 32.2 mm
- net -4V_A: track 305.0 -> 284.0 mm, vias 9 -> 11
- net /Analog Rails/5V_OK: track 122.3 -> 142.7 mm, vias 2 -> 4
- net /Controller/PWR_GOOD: track 183.8 -> 202.9 mm, vias 3 -> 4
- net Net-(RN10-R3.1): track 2.78 -> 20.7 mm, vias 0 -> 2
- net /Path Switching/LDO_OUT: track 41.2 -> 23.7 mm, vias 2 -> 32
- net /Controller/GATE_AMP: track 145.4 -> 162.9 mm
- net +5V: track 322.1 -> 337.6 mm, vias 7 -> 20
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- added copper zone on F.Cu, net +12V_A
- added copper zone on F.Cu, net +13V5
- added copper zone on F.Cu, net +5V
- added copper zone on In2.Cu, net +5V
- added copper zone on B.Cu, net /Monitors/VIN_P
- added copper zone on F.Cu, net /Monitors/VIN_P
- added copper zone on B.Cu, net /Monitors/VOUT_BUF
- added copper zone on F.Cu, net /Monitors/VOUT_BUF
- added copper zone on F.Cu, net /Output Stage/VIN_RAW
- added copper zone on F.Cu, net /Output Stage/VOUT_S
- added copper zone on B.Cu, net /Path Switching/LDO_OUT
- added copper zone on F.Cu, net /Path Switching/LDO_OUT
- added copper zone on B.Cu, net /Path Switching/SUPPLY
- added copper zone on F.Cu, net /Path Switching/SUPPLY
- added copper zone on B.Cu, net GND
- added copper zone on F.Cu, net GND
- added copper zone on In2.Cu, net GND
- added copper zone on B.Cu, net Net-(C42-Pad1)
- added copper zone on F.Cu, net Net-(C42-Pad1)
- added copper zone on F.Cu, net Net-(D11-K)
- added copper zone on F.Cu, net Net-(D18-A)
- added copper zone on F.Cu, net Net-(D19-A)
- added copper zone on F.Cu, net Net-(D21-K)
- added copper zone on F.Cu, net Net-(D6-A)
- added copper zone on F.Cu, net Net-(L2-Pad1)
- added copper zone on F.Cu, net Net-(L2-Pad2)
- added copper zone on F.Cu, net Net-(Q14-S-Pad1)
- added copper zone on F.Cu, net Net-(Q15-S-Pad1)
Other:
- board text added: "Open Power Profiler - Carrier Board rev A2 draft"
- board text removed: "Power Profiler - Carrier Board rev A2 draft"
